Commit message: feat(urdf): adding a most recent urdf export

File: src/amr_description/urdf/amr.urdf (robot description, URDF)
Before this commit: robot amr, 2 links, 1 joints
Links:
- added link back_pitch_link
- added link back_roll_link
- added link back_yaw_link
- added link front_pitch_link
- added link front_roll_link
- added link front_yaw_link
- added link left_wheel
- added link right_wheel
Joints:
- added joint back_pitch_joint: type fixed, parent back_roll_link, child back_pitch_link
- added joint back_roll_joint: type fixed, parent back_yaw_link, child back_roll_link
- added joint back_yaw_joint: type fixed, parent chassis, child back_yaw_link
- added joint front_pitch_joint: type fixed, parent front_roll_link, child front_pitch_link
- added joint front_roll_joint: type fixed, parent front_yaw_link, child front_roll_link
- added joint front_yaw_joint: type fixed, parent chassis, child front_yaw_link
- added joint joint_left_wheel: type continuous, parent chassis, child left_wheel
- added joint joint_rigth_wheel: type continuous, parent chassis, child rigth_wheel
